File: kicad-template/USB-Micro.sch (KiCad schematic (older format))
At the start: 2 parts

Commit message: working on adding support for jlcpcb small batch assembly
Parts:
- ESD1: LCSC (none) -> C12333
- USB1: LCSC (none) -> C132562
Changed lines of the file:
@@
 F 6 "Amphenol" H 3225 3175 50  0001 C CNN "Manufactuer"
 F 7 "USB Connectors 5P MICRO USB TYPE B RECEPTACLE W/ PEGS" H 3225 3175 50  0001 C CNN "Description"
+F 8 "C132562" H 3225 3175 50  0001 C CNN "LCSC"
 	1    3225 3175
 	1    0    0    -1
@@
 F 7 "Nexperia" H 2300 -1675 50  0001 C CNN "Manufacturer"
 F 8 "PRTR5V0U2X,215	" H 0   0   50  0001 C CNN "Seeed Part Num"
+F 9 "C12333" H 7100 3475 50  0001 C CNN "LCSC"
 	1    7100 3475
 	1    0    0    -1
