File: kicad-template/USB-Support.sch (KiCad schematic (older format))
At the start: 11 parts

Commit message: working on adding support for jlcpcb small batch assembly
Parts:
- C10, C9: LCSC (none) -> C277499
- C11: LCSC (none) -> C107135
- C12, C13: LCSC (none) -> C107045
- L1: LCSC (none) -> C88995
- R3: LCSC (none) -> C131054
- R4, R5: LCSC (none) -> C107701
- RV1, RV2: LCSC (none) -> C118414
Changed lines of the file:
@@
 $Descr A4 11693 8268
 encoding utf-8
-Sheet 6 13
+Sheet 8 13
 Title ""
 Date "2016-05-06"
@@
 F 7 "BLM31PG391SN1L" H 2100 5000 60  0001 C CNN "MPN"
 F 8 "BLM31PG391SN1L" H 0   0   50  0001 C CNN "Seeed Part Num"
+F 9 "C88995" V 2100 5000 50  0001 C CNN "LCSC"
 	1    2100 5000
 	0    1    1    0
@@
 F 7 "RES SMD 22 OHM 1% 1/10W 0603" V 7025 4575 60  0001 C CNN "Description"
 F 8 "RC0603FR-0722RL	" H 0   0   50  0001 C CNN "Seeed Part Num"
+F 9 "C107701" V 7025 4575 50  0001 C CNN "LCSC"
 	1    7025 4575
 	0    -1   1    0
@@
 F 7 "311-22.0HRTR-ND" V 7050 5200 60  0001 C CNN "DigiKey"
 F 8 "RC0603FR-0722RL	" H 0   0   50  0001 C CNN "Seeed Part Num"
+F 9 "C107701" V 7050 5200 50  0001 C CNN "LCSC"
 	1    7050 5200
 	0    -1   1    0
@@
 AR Path="/5B90A59F/5CA5B290/566B7A90" Ref="#PWR?"  Part="1"
 AR Path="/5CA5B290/566B7A90" Ref="#PWR?"  Part="1"
+AR Path="/5D950BDF/5CA5B290/566B7A90" Ref="#PWR?"  Part="1"
 F 0 "#PWR?" H 2450 5300 30  0001 C CNN
 F 1 "GND" H 2450 5250 30  0001 C CNN
@@
 AR Path="/5B90A59F/5CA5B290/5667E4FB" Ref="#PWR?"  Part="1"
 AR Path="/5CA5B290/5667E4FB" Ref="#PWR?"  Part="1"
+AR Path="/5D950BDF/5CA5B290/5667E4FB" Ref="#PWR?"  Part="1"
 F 0 "#PWR?" H 1750 5300 30  0001 C CNN
 F 1 "GND" H 1750 5250 30  0001 C CNN
@@
 AR Path="/5B90A59F/5CA5B290/56760E65" Ref="#PWR?"  Part="1"
 AR Path="/5CA5B290/56760E65" Ref="#PWR?"  Part="1"
+AR Path="/5D950BDF/5CA5B290/56760E65" Ref="#PWR?"  Part="1"
 F 0 "#PWR?" H 3300 4600 50  0001 C CNN
 F 1 "+5V" H 3300 4890 50  0000 C CNN
@@
 F 7 "CAP CER 4.7UF 16V X7R 0805" H -175 75  50  0001 C CNN "Description"
 F 8 "CL21B475KOFNNNE" H 0   0   50  0001 C CNN "Seeed Part Num"
+F 9 "C277499" H 2450 5150 50  0001 C CNN "LCSC"
 	1    2450 5150
 	1    0    0    -1
@@
 F 7 "CAP CER 4.7UF 16V X7R 0805" H -875 -625 50  0001 C CNN "Description"
 F 8 "CL21B475KOFNNNE" H 0   0   50  0001 C CNN "Seeed Part Num"
+F 9 "C277499" H 1750 5150 50  0001 C CNN "LCSC"
 	1    1750 5150
 	1    0    0    -1
@@
 F 7 "Yaego" H 0   0   50  0001 C CNN "Manufacturer"
 F 8 "CC0603JRNPO9BN270	" H 0   0   50  0001 C CNN "Seeed Part Num"
+F 9 "C107045" H 6750 5300 50  0001 C CNN "LCSC"
 	1    6750 5300
 	1    0    0    -1
@@
 AR Path="/5B90A59F/5CA5B290/5FD0B119" Ref="#PWR?"  Part="1"
 AR Path="/5CA5B290/5FD0B119" Ref="#PWR?"  Part="1"
+AR Path="/5D950BDF/5CA5B290/5FD0B119" Ref="#PWR?"  Part="1"
 F 0 "#PWR?" H 6750 5450 30  0001 C CNN
 F 1 "VSS" H 6750 5380 30  0000 C CNN
@@
 AR Path="/5B90A59F/5CA5B290/5C679C8B" Ref="#PWR?"  Part="1"
 AR Path="/5CA5B290/5C679C8B" Ref="#PWR?"  Part="1"
+AR Path="/5D950BDF/5CA5B290/5C679C8B" Ref="#PWR?"  Part="1"
 F 0 "#PWR?" H 6750 4825 30  0001 C CNN
 F 1 "VSS" H 6750 4755 30  0000 C CNN
@@
 AR Path="/5B90A59F/5CA5B290/5B5FB123" Ref="#PWR?"  Part="1"
 AR Path="/5CA5B290/5B5FB123" Ref="#PWR?"  Part="1"
+AR Path="/5D950BDF/5CA5B290/5B5FB123" Ref="#PWR?"  Part="1"
 F 0 "#PWR?" H 3975 7050 30  0001 C CNN
 F 1 "VSS" H 3975 6980 30  0000 C CNN
@@
 F 7 "CAP CER 10000PF 100V X7R 0805" H 3825 6500 60  0001 C CNN "Description"
 F 8 "GCM21BR72A104KA37L	" H 0   0   50  0001 C CNN "Seeed Part Num"
+F 9 "C107135" H 3825 6500 50  0001 C CNN "LCSC"
 	1    3825 6500
 	1    0    0    -1
@@
 F 7 "Yaego" H 2625 3750 50  0001 C CNN "Manufacturer"
 F 8 "RC0603FR-07499KL	" H 0   0   50  0001 C CNN "Seeed Part Num"
+F 9 "C131054" H 4125 6550 50  0001 C CNN "LCSC"
 	1    4125 6550
 	1    0    0    -1
@@
 F 7 "Yaego" H -125 -250 50  0001 C CNN "Manufacturer"
 F 8 "CC0603JRNPO9BN270	" H 0   0   50  0001 C CNN "Seeed Part Num"
+F 9 "C107045" H 6750 4675 50  0001 C CNN "LCSC"
 	1    6750 4675
 	1    0    0    -1
@@
 F 6 "F3363CT-ND" H 0   0   50  0001 C CNN "DigiKey"
 F 7 "V5.5MLA0603NH" H 0   0   50  0001 C CNN "MPN"
+F 8 "C118414" V 2125 6125 50  0001 C CNN "LCSC"
 	1    2125 6125
 	0    1    1    0
@@
 F 6 "F3363CT-ND" H 0   0   50  0001 C CNN "DigiKey"
 F 7 "V5.5MLA0603NH" H 0   0   50  0001 C CNN "MPN"
+F 8 "C118414" V 2125 6600 50  0001 C CNN "LCSC"
 	1    2125 6600
 	0    1    1    0
