File: kicad-template/MCU-ATmega32u4.sch (KiCad schematic (older format))
At the start: 25 parts, among them J1 ICSP, SW1 SW_PUSH, T5 ICSP_Test, U1 ATMEGA32U4-MU, X1 ABM3-16.000

Commit message: working on adding support for jlcpcb small batch assembly
Parts:
- C1, C2, C3, C4, C6: LCSC (none) -> C106214
- C5, C7: LCSC (none) -> C107045
- D2: LCSC (none) -> C83528
- R1: LCSC (none) -> C130232
- R2: DigiKey RG16P3.3KBCT-ND -> 311-330GRTR-ND; LCSC (none) -> C105879; MPN RG1608P-332-B-T5 -> 311-330GRTR-ND; Manufacturer Susumu -> Yaego
- X1: value ABM3-16.000 -> 16Mhz-18pF; footprint Keyboardio:ABM3_Crystal_Oscillator -> Crystal:Crystal_SMD_SeikoEpson_TSX3225-4Pin_3.2x2.5mm; symbol Device:Crystal -> Device:Crystal_GND24; Description Crystal 16.0000MHz 20ppm 18pF 40 Ohm -40°C - 85°C Surface M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 -> SMD Crystal Resonators 16MHz ±10ppm TSX-3225 RoHS 18pf; DigiKey http://www.digikey.com/product-detail/en/ABM3-16.000MHZ-D2Y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 -> TSX-322516.0000MF20G-C-ND; LCSC (none) -> C255907; MPN ABM3-16.000MHZ-D2Y-T -> X1E000021069600; Manufacturer Abracon -> Seiko-Epson
Connections:
- net GND: now also X1.2, X1.4
- net at C5.1, U1.17 (XTAL1), XTAL1.1: now also X1.3; no longer X1.2
Changed lines of the file:
@@
 F 7 "CAP CER 27PF 50V C0G/NP0 0603" H 2750 5300 60  0001 C CNN "Description"
 F 8 "CC0603JRNPO9BN270	" H 0   0   50  0001 C CNN "Seeed Part Num"
+F 9 "C107045" H 2750 5300 50  0001 C CNN "LCSC"
 	1    2750 5300
 	1    0    0    -1
@@
 F 7 "RES SMD 10K OHM 0.5% 1/16W 0603" V 8400 3100 60  0001 C CNN "Description"
 F 8 "RK73H1JTTD1002F" H 0   0   50  0001 C CNN "Seeed Part Num"
+F 9 "C130232" V 8400 3100 50  0001 C CNN "LCSC"
 	1    8400 3100
 	-1   0    0    1
@@
 F 7 "CAP CER 27PF 50V C0G/NP0 0603" H 3500 5300 60  0001 C CNN "Description"
 F 8 "CC0603JRNPO9BN270	" H 0   0   50  0001 C CNN "Seeed Part Num"
+F 9 "C107045" H 3500 5300 50  0001 C CNN "LCSC"
 	1    3500 5300
 	1    0    0    -1
@@
 F 7 "CC0603KRX5R6BB105" H 1800 3675 60  0001 C CNN "MPN"
 F 8 "GRM188R61A105KA61D	" H 0   0   50  0001 C CNN "Seeed Part Num"
+F 9 "C106214" H 1800 3675 50  0001 C CNN "LCSC"
 	1    1800 3675
 	0    -1   1    0
@@
 F 7 "CC0603KRX5R6BB105" H 1800 3325 60  0001 C CNN "MPN"
 F 8 "GRM188R61A105KA61D	" H 0   0   50  0001 C CNN "Seeed Part Num"
+F 9 "C106214" H 1800 3325 50  0001 C CNN "LCSC"
 	1    1800 3325
 	0    -1   1    0
@@
 F 7 "CC0603KRX5R6BB105" H 3400 4150 60  0001 C CNN "MPN"
 F 8 "GRM188R61A105KA61D	" H 0   0   50  0001 C CNN "Seeed Part Num"
+F 9 "C106214" H 3400 4150 50  0001 C CNN "LCSC"
 	1    3400 4150
 	-1   0    0    -1
@@
 F 6 "1N4148W-7-F" H 6950 1250 60  0001 C CNN "MPN"
 F 7 "DIODE GEN PURP 100V 300MA SOD123" H 6950 1250 60  0001 C CNN "Description"
+F 8 "C83528" H 8700 3050 50  0001 C CNN "LCSC"
 	1    8700 3050
 	0    1    1    0
@@
 F 1 "330R 5%" V 9100 4000 40  0000 C CNN
 F 2 "Resistor_SMD:R_0603_1608Metric" V 9130 4000 30  0001 C CNN
-F 3 "https://media.digikey.com/pdf/Data%20Sheets/Susumu%20PDFs/RG_RM_RGH_Oct2012.pdf" H 9200 4000 30  0001 C CNN
+F 3 "http://www.yageo.com/documents/recent/PYu-RC_Group_51_RoHS_L_10.pdf" H 9200 4000 30  0001 C CNN
 F 4 "RES SMD 330 OHM 5% 1/10W 0603" H -3975 -100 50  0001 C CNN "Description"
-F 5 "RG16P3.3KBCT-ND" H -3975 -100 50  0001 C CNN "DigiKey"
-F 6 "RG1608P-332-B-T5" H -3975 -100 50  0001 C CNN "MPN"
-F 7 "Susumu" H -3975 -100 50  0001 C CNN "Manufacturer"
+F 5 "311-330GRTR-ND" H -3975 -100 50  0001 C CNN "DigiKey"
+F 6 "311-330GRTR-ND" H -3975 -100 50  0001 C CNN "MPN"
+F 7 "Yaego" H -3975 -100 50  0001 C CNN "Manufacturer"
 F 8 "RC0603JR-07330RL" H 0   0   50  0001 C CNN "Seeed Part Num"
+F 9 "C105879" V 9200 4000 50  0001 C CNN "LCSC"
 	1    9200 4000
 	0    -1   -1   0
@@
 F 7 "CC0603KRX5R6BB105" H 1800 2975 60  0001 C CNN "MPN"
 F 8 "GRM188R61A105KA61D	" H 0   0   50  0001 C CNN "Seeed Part Num"
+F 9 "C106214" H 1800 2975 50  0001 C CNN "LCSC"
 	1    1800 2975
 	0    -1   1    0
@@
 F 7 "CC0603KRX5R6BB105" H 1800 4025 60  0001 C CNN "MPN"
 F 8 "GRM188R61A105KA61D	" H 0   0   50  0001 C CNN "Seeed Part Num"
+F 9 "C106214" H 1800 4025 50  0001 C CNN "LCSC"
 	1    1800 4025
 	0    -1   1    0
@@
 $EndComp
 Wire Wire Line
-	3650 5050 3650 4750
-Wire Wire Line
-	3650 4750 2750 4750
-Wire Wire Line
-	2750 4750 2750 5050
+	3650 5050 3650 4575
+Wire Wire Line
+	3650 4575 2750 4575
+Wire Wire Line
+	2750 4575 2750 5050
 Text GLabel 6100 5250 2    50   Input ~ 0
 COL16
@@
 	8850 3650 8950 3650
 $Comp
-L Device:Crystal X1
+L Device:Crystal_GND24 X1
 U 1 1 545C2706
 P 3050 5150
-F 0 "X1" H 3050 5300 60  0000 C CNN
-F 1 "ABM3-16.000" H 2975 4950 60  0000 C CNN
-F 2 "Keyboardio:ABM3_Crystal_Oscillator" H 3050 5150 60  0001 C CNN
-F 3 "http://www.abracon.com/Resonators/abm3.pdf" H 3050 5150 60  0001 C CNN
-F 4 "Abracon" H 3050 5150 60  0001 C CNN "Manufacturer"
-F 5 "ABM3-16.000MHZ-D2Y-T" H 3050 5150 60  0001 C CNN "MPN"
-F 6 "http://www.digikey.com/product-detail/en/ABM3-16.000MHZ-D2Y-T/535-10638-2-ND/2344578" H 3050 5150 60  0001 C CNN "DigiKey"
-F 7 "Crystal 16.0000MHz 20ppm 18pF 40 Ohm -40°C - 85°C Surface Mount 2-SMD" H 3050 5150 60  0001 C CNN "Description"
+F 0 "X1" H 2875 5250 60  0000 C CNN
+F 1 "16Mhz-18pF" H 2975 4950 60  0000 C CNN
+F 2 "Crystal:Crystal_SMD_SeikoEpson_TSX3225-4Pin_3.2x2.5mm" H 3050 5150 60  0001 C CNN
+F 3 "https://support.epson.biz/td/api/doc_check.php?dl=brief_TSX-3225&lang=en" H 3050 5150 60  0001 C CNN
+F 4 "Seiko-Epson" H 3050 5150 60  0001 C CNN "Manufacturer"
+F 5 "X1E000021069600" H 3050 5150 60  0001 C CNN "MPN"
+F 6 "TSX-322516.0000MF20G-C-ND" H 3050 5150 60  0001 C CNN "DigiKey"
+F 7 "SMD Crystal Resonators 16MHz ±10ppm TSX-3225 RoHS 18pf" H 3050 5150 50  0001 C CNN "Description"
+F 8 "C255907" H 3050 5150 50  0001 C CNN "LCSC"
 	1    3050 5150
 	-1   0    0    1
@@
 Text GLabel 6100 4850 2    50   Input ~ 0
 COL8
+$Comp
+L Keyboard-symbols:GND #PWR?
+U 1 1 5D998C9C
+P 3050 5400
+F 0 "#PWR?" H 3050 5150 50  0001 C CNN
+F 1 "GND" H 3055 5227 50  0000 C CNN
+F 2 "" H 3050 5400 50  0000 C CNN
+F 3 "" H 3050 5400 50  0000 C CNN
+	1    3050 5400
+	1    0    0    -1
+$EndComp
+$Comp
+L Keyboard-symbols:GND #PWR?
+U 1 1 5D9999E0
+P 3050 4875
+F 0 "#PWR?" H 3050 4625 50  0001 C CNN
+F 1 "GND" H 3055 4702 50  0000 C CNN
+F 2 "" H 3050 4875 50  0000 C CNN
+F 3 "" H 3050 4875 50  0000 C CNN
+	1    3050 4875
+	-1   0    0    1
+$EndComp
+Wire Wire Line
+	3050 4875 3050 4950
+Wire Wire Line
+	3050 5400 3050 5350
 $EndSCHEMATC

Commit message: snapshot changes
Other:
- moved on the sheet: AREF1, C5, C6, C7, C8, D2, J1, LED_DRIVER_INTB1, LED_DRIVER_SDB1, R1, R2, SCL1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
