File: normal-60/normal-60.kicad_pcb (KiCad board)
At the start: 2 copper layers, 284.3 x 116.2 mm, 152 parts, among them J1 ICSP, SW1 SW_PUSH, U1 ATMEGA32U4-MU, X1 16Mhz-18pF

Commit message: snapshot changes
Parts:
- moved L1 3.74 mm to (133.2, 141.8)
- moved C9 3.73 mm to (133.8, 139.6)
- moved C10 2.14 mm to (126.9, 141.6)
- moved C12 2.11 mm to (129.4, 141.8)
- moved C13 2.11 mm to (129.4, 137.3)
- moved R4 2.11 mm to (129.4, 140.3)
- moved R5 2.11 mm to (129.4, 138.8)
- moved C2 0.32 mm to (125.1, 141.8), turned to 90 degrees
- moved C7 0.24 mm to (123.1, 131.8)
- moved X1 0.23 mm to (120.2, 132.1)
- moved C3 0.19 mm to (115.7, 131.8)
- moved C5 0.14 mm to (117.3, 131.8)
Routing:
- net COL7: track 149.9 -> 142.1 mm
- net COL9: track 109.8 -> 104.3 mm
- net ROW4: track 308.9 -> 313.1 mm
- net USB_D+: track 106.9 -> 103.7 mm
- net +5V: track 84.0 -> 87.3 mm, vias 7 -> 8
- net USB_D-: track 107.5 -> 104.3 mm
- net R_D+: track 8.08 -> 5.74 mm
- net USBVBUS: track 112.0 -> 109.7 mm
- net GND: track 54.4 -> 56.7 mm, vias 53 -> 46
- net COL1: track 251.5 -> 249.3 mm
- net COL12: track 173.0 -> 171.4 mm, vias 6 -> 4
- net ROW3: track 329.3 -> 327.8 mm
- net R_D-: track 8.38 -> 6.85 mm
- net COL11: track 159.2 -> 157.8 mm, vias 8 -> 6
- net COL10: track 135.8 -> 134.5 mm, vias 8 -> 6
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